File: _autosave-usbsplitter.kicad_sch (KiCad schematic)
At the start: 7 parts, among them SW1 SW_SPDT, SW2 SW_SPDT, SW3 SW_SPDT, SW4 SW_SPDT

Commit message: v1.0.0
Parts:
- renumbered IN to IN1
Changed lines of the file:
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@@
   (symbol (lib_id "Connector:USB_A") (at 111.76 82.55 270) (unit 1)
     (in_bom yes) (on_board yes) (dnp no) (fields_autoplaced)
-    (property "Reference" "IN" (at 120.65 81.915 90)
+    (property "Reference" "IN1" (at 120.65 81.915 90)
       (effects (font (size 1.27 1.27)) (justify left))
     )
@@
       (project "usbsplitter"
         (path "/762276e9-b28b-4427-9958-3dbb372bff80"
-          (reference "IN") (unit 1)
+          (reference "IN1") (unit 1)
         )
       )
