File: usbsplitter.kicad_pcb (KiCad board)
At the start: 2 copper layers, 49 x 38 mm, 11 parts, among them SW1 SW_SPDT, SW2 SW_SPDT, SW3 SW_SPDT, SW4 SW_SPDT

Commit message: v1.0.1
Parts:
- moved SW1 2.00 mm to (179.0, 70.0)
- moved SW3 1.00 mm to (179.0, 74.0)
- moved SW4 1.00 mm to (179.0, 82.0)
Routing:
- net +5V: track 54.9 -> 44.7 mm
- net GND: track 22.6 -> 23.6 mm
- net /5VA: track 20.4 -> 19.5 mm
- net /5VB: track 15.2 -> 14.4 mm
Other:
- board text added: "2023-04"
- board text added: "ndelucca usbsplitter v1.0.1"
- board text removed: "ndelucca usbsplitter v1.0"
Changed lines of the file:
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@@
   )
   (footprint "Connector_PinHeader_2.54mm:PinHeader_1x03_P2.54mm_Vertical" (layer "F.Cu")
-    (at 179 73 -90)
+    (at 179 74 -90)
     (descr "Through hole straight pin header, 1x03, 2.54mm pitch, single row")
     (tags "Through hole pin header THT 1x03 2.54mm single row")
@@
   )
   (footprint "Connector_PinHeader_2.54mm:PinHeader_1x03_P2.54mm_Vertical" (layer "F.Cu")
-    (at 179 83 -90)
+    (at 179 82 -90)
     (descr "Through hole straight pin header, 1x03, 2.54mm pitch, single row")
     (tags "Through hole pin header THT 1x03 2.54mm single row")
@@
   )
   (footprint "Connector_PinHeader_2.54mm:PinHeader_1x03_P2.54mm_Vertical" (layer "F.Cu")
-    (at 179 68 -90)
+    (at 179 70 -90)
     (descr "Through hole straight pin header, 1x03, 2.54mm pitch, single row")
     (tags "Through hole pin header THT 1x03 2.54mm single row")
@@
   (gr_line (start 201 65) (end 152 65)
     (stroke (width 0.1) (type default)) (layer "Edge.Cuts"))
-  (gr_text "ndelucca\nusbsplitter\nv1.0" (at 156 95) (layer "F.SilkS")
+  (gr_text "2023-04" (at 186 102) (layer "F.SilkS")
     (effects (font (size 1 1) (thickness 0.15)) (justify left bottom))
   )
-  (segment (start 175.37 66.55) (end 161.45 66.55) (width 0.8) (layer "F.Cu") (net 1))
-  (segment (start 172.5 87.5) (end 172.5 88.2725) (width 0.8) (layer "F.Cu") (net 1))
-  (segment (start 176.46 67.64) (end 175.37 66.55) (width 0.8) (layer "F.Cu") (net 1))
-  (segment (start 153 77.910902) (end 157.881991 82.792893) (width 0.8) (layer "F.Cu") (net 1))
-  (segment (start 161.45 66.55) (end 153 75) (width 0.8) (layer "F.Cu") (net 1))
-  (segment (start 176.46 68) (end 176.46 67.64) (width 0.8) (layer "F.Cu") (net 1))
-  (segment (start 167.792893 82.792893) (end 172.5 87.5) (width 0.8) (layer "F.Cu") (net 1))
-  (segment (start 157.881991 82.792893) (end 167.792893 82.792893) (width 0.8) (layer "F.Cu") (net 1))
-  (segment (start 153 75) (end 153 77.910902) (width 0.8) (layer "F.Cu") (net 1))
-  (segment (start 171.47 77.99) (end 171.47 84.7425) (width 0.8) (layer "F.Cu") (net 2))
+  (gr_text "ndelucca\nusbsplitter v1.0.1" (at 153 94) (layer "F.SilkS")
+    (effects (font (size 1 1) (thickness 0.15)) (justify left bottom))
+  )
+  (segment (start 157.138 80.291659) (end 157.138 78.862) (width 0.8) (layer "F.Cu") (net 1))
+  (segment (start 157.138 78.862) (end 168 68) (width 0.8) (layer "F.Cu") (net 1))
+  (segment (start 167.020393 82.792893) (end 159.639234 82.792893) (width 0.8) (layer "F.Cu") (net 1))
+  (segment (start 172.5 88.2725) (end 167.020393 82.792893) (width 0.8) (layer "F.Cu") (net 1))
+  (segment (start 174.46 68) (end 176.46 70) (width 0.8) (layer "F.Cu") (net 1))
+  (segment (start 168 68) (end 174.46 68) (width 0.8) (layer "F.Cu") (net 1))
+  (segment (start 159.639234 82.792893) (end 157.138 80.291659) (width 0.8) (layer "F.Cu") (net 1))
   (segment (start 171.47 84.7425) (end 175 88.2725) (width 0.8) (layer "F.Cu") (net 2))
-  (segment (start 176.46 73) (end 171.47 77.99) (width 0.8) (layer "F.Cu") (net 2))
-  (segment (start 172.47 81.99) (end 172.47 83.7425) (width 0.8) (layer "F.Cu") (net 3))
-  (segment (start 176.46 78) (end 172.47 81.99) (width 0.8) (layer "F.Cu") (net 3))
-  (segment (start 172.47 83.7425) (end 177 88.2725) (width 0.8) (layer "F.Cu") (net 3))
+  (segment (start 175.01 75.45) (end 176.46 74) (width 0.8) (layer "F.Cu") (net 2))
+  (segment (start 171.47 84.7425) (end 171.47 77.53) (width 0.8) (layer "F.Cu") (net 2))
+  (segment (start 173.55 75.45) (end 175.01 75.45) (width 0.8) (layer "F.Cu") (net 2))
+  (segment (start 171.47 77.53) (end 173.55 75.45) (width 0.8) (layer "F.Cu") (net 2))
+  (segment (start 172.47 81.39939) (end 173.86939 80) (width 0.8) (layer "F.Cu") (net 3))
+  (segment (start 172.47 83.7425) (end 172.47 81.39939) (width 0.8) (layer "F.Cu") (net 3))
+  (segment (start 174.46 80) (end 176.46 78) (width 0.8) (layer "F.Cu") (net 3))
+  (segment (start 177 88.2725) (end 172.47 83.7425) (width 0.8) (layer "F.Cu") (net 3))
+  (segment (start 173.86939 80) (end 174.46 80) (width 0.8) (layer "F.Cu") (net 3))
   (segment (start 179 90.9825) (end 182.57 90.9825) (width 0.8) (layer "F.Cu") (net 4))
   (segment (start 169.43 90.9825) (end 179 90.9825) (width 0.8) (layer "F.Cu") (net 4))
   (segment (start 179.5 90.4825) (end 179 90.9825) (width 0.8) (layer "F.Cu") (net 4))
-  (segment (start 176.46 83) (end 176.46 85.2325) (width 0.8) (layer "F.Cu") (net 4))
   (segment (start 179.5 88.2725) (end 179.5 90.4825) (width 0.8) (layer "F.Cu") (net 4))
+  (segment (start 176.46 85.2325) (end 176.46 82) (width 0.8) (layer "F.Cu") (net 4))
   (segment (start 176.46 85.2325) (end 179.5 88.2725) (width 0.8) (layer "F.Cu") (net 4))
-  (segment (start 179 68) (end 182.7725 68) (width 0.8) (layer "F.Cu") (net 5))
-  (segment (start 182.7725 68) (end 194.5 79.7275) (width 0.8) (layer "F.Cu") (net 5))
-  (segment (start 186.35013 73) (end 192 78.64987) (width 0.8) (layer "B.Cu") (net 6))
-  (segment (start 179 73) (end 186.35013 73) (width 0.8) (layer "B.Cu") (net 6))
+  (segment (start 184.7725 70) (end 187.88625 73.11375) (width 0.8) (layer "F.Cu") (net 5))
+  (segment (start 187.88625 73.11375) (end 194.5 79.7275) (width 0.8) (layer "F.Cu") (net 5))
+  (segment (start 179 70) (end 184.7725 70) (width 0.8) (layer "F.Cu") (net 5))
   (segment (start 192 78.64987) (end 192 79.7275) (width 0.8) (layer "B.Cu") (net 6))
+  (segment (start 187.01763 73.6675) (end 179.3325 73.6675) (width 0.8) (layer "B.Cu") (net 6))
+  (segment (start 179.3325 73.6675) (end 179 74) (width 0.8) (layer "B.Cu") (net 6))
+  (segment (start 192 78.64987) (end 187.01763 73.6675) (width 0.8) (layer "B.Cu") (net 6))
+  (segment (start 182.3325 74.6675) (end 179 78) (width 0.8) (layer "B.Cu") (net 7))
+  (segment (start 186.01763 74.6675) (end 182.3325 74.6675) (width 0.8) (layer "B.Cu") (net 7))
   (segment (start 190 78.64987) (end 190 79.7275) (width 0.8) (layer "B.Cu") (net 7))
   (segment (start 186.01763 74.6675) (end 190 78.64987) (width 0.8) (layer "B.Cu") (net 7))
-  (segment (start 182.3325 74.6675) (end 186.01763 74.6675) (width 0.8) (layer "B.Cu") (net 7))
-  (segment (start 179 78) (end 182.3325 74.6675) (width 0.8) (layer "B.Cu") (net 7))
+  (segment (start 179 82) (end 185.2275 82) (width 0.8) (layer "B.Cu") (net 8))
   (segment (start 185.61375 81.61375) (end 187.5 79.7275) (width 0.8) (layer "B.Cu") (net 8))
   (segment (start 184.43 80.43) (end 185.61375 81.61375) (width 0.8) (layer "B.Cu") (net 8))
   (segment (start 185.61375 81.61375) (end 195.448623 81.61375) (width 0.8) (layer "B.Cu") (net 8))
   (segment (start 197.57 79.492373) (end 197.57 77.0175) (width 0.8) (layer "B.Cu") (net 8))
+  (segment (start 185.2275 82) (end 185.61375 81.61375) (width 0.8) (layer "B.Cu") (net 8))
   (segment (start 195.448623 81.61375) (end 197.57 79.492373) (width 0.8) (layer "B.Cu") (net 8))
-  (segment (start 184.2275 83) (end 185.61375 81.61375) (width 0.8) (layer "B.Cu") (net 8))
   (segment (start 184.43 77.0175) (end 184.43 80.43) (width 0.8) (layer "B.Cu") (net 8))
-  (segment (start 179 83) (end 184.2275 83) (width 0.8) (layer "B.Cu") (net 8))
-  (segment (start 173.92 68) (end 165.5 76.42) (width 0.8) (layer "F.Cu") (net 9))
+  (segment (start 171.92 70) (end 170.46 71.46) (width 0.8) (layer "F.Cu") (net 9))
   (segment (start 165.5 76.42) (end 165.5 79.7275) (width 0.8) (layer "F.Cu") (net 9))
-  (segment (start 168.64987 73) (end 173.92 73) (width 0.8) (layer "B.Cu") (net 10))
-  (segment (start 163 78.64987) (end 168.64987 73) (width 0.8) (layer "B.Cu") (net 10))
+  (segment (start 173.92 70) (end 171.92 70) (width 0.8) (layer "F.Cu") (net 9))
+  (segment (start 170.46 71.46) (end 165.5 76.42) (width 0.8) (layer "F.Cu") (net 9))
+  (segment (start 167.64987 74) (end 173.92 74) (width 0.8) (layer "B.Cu") (net 10))
+  (segment (start 163 78.64987) (end 167.64987 74) (width 0.8) (layer "B.Cu") (net 10))
   (segment (start 163 79.7275) (end 163 78.64987) (width 0.8) (layer "B.Cu") (net 10))
   (segment (start 162.8225 81.55) (end 170.37 81.55) (width 0.8) (layer "B.Cu") (net 11))
-  (segment (start 170.37 81.55) (end 173.92 78) (width 0.8) (layer "B.Cu") (net 11))
+  (segment (start 173.92 78) (end 170.37 81.55) (width 0.8) (layer "B.Cu") (net 11))
   (segment (start 161 79.7275) (end 162.8225 81.55) (width 0.8) (layer "B.Cu") (net 11))
-  (segment (start 155.43 77.0175) (end 155.79 77.0175) (width 0.8) (layer "F.Cu") (net 12))
   (segment (start 168.57 77.0175) (end 168.57 79.492373) (width 0.8) (layer "F.Cu") (net 12))
-  (segment (start 155.79 77.0175) (end 158.5 79.7275) (width 0.8) (layer "F.Cu") (net 12))
   (segment (start 160.565393 81.792893) (end 158.5 79.7275) (width 0.8) (layer "F.Cu") (net 12))
   (segment (start 166.26948 81.792893) (end 160.565393 81.792893) (width 0.8) (layer "F.Cu") (net 12))
   (segment (start 168.57 79.492373) (end 166.26948 81.792893) (width 0.8) (layer "F.Cu") (net 12))
+  (segment (start 155.79 77.0175) (end 158.5 79.7275) (width 0.8) (layer "B.Cu") (net 12))
+  (segment (start 161.7725 83) (end 172.92 83) (width 0.8) (layer "B.Cu") (net 12))
   (segment (start 158.5 79.7275) (end 161.7725 83) (width 0.8) (layer "B.Cu") (net 12))
-  (segment (start 161.7725 83) (end 173.92 83) (width 0.8) (layer "B.Cu") (net 12))
+  (segment (start 155.43 77.0175) (end 155.79 77.0175) (width 0.8) (layer "B.Cu") (net 12))
+  (segment (start 172.92 83) (end 173.92 82) (width 0.8) (layer "B.Cu") (net 12))
   (zone (net 4) (net_name "GND") (layer "F.Cu") (hatch edge 0.5)
     (connect_pads (clearance 0.5))
